Commit message: joey moment

File: src/scorpio/description/lidar.xacro (robot description, xacro)
@@ -4,5 +4,6 @@
         <parent link="chassis"/>
         <child link="laser_frame"/>
-        <origin xyz="0.3175 0 0.12" rpy="0 1.5707 0"/>
+        <origin xyz="0.3175 0 0.12" rpy="0 1.5708 0"/>
+		<!-- <origin xyz="0.3175 0 0.12" rpy="0 1.5707 0"/>-->
     </joint>
     <link name="laser_frame">

File: src/scorpio/description/robot_core.xacro (robot description, xacro)
@@ -50,5 +50,5 @@
     </gazebo>
     <!-- LEFT FRONT WHEEL LINK -->
-    <joint name="left_front_wheel_joint" type="continuous">
+    <joint name="left_front_wheel_joint" type="fixed">
         <parent link="base_link"/>
         <child link="left_front_wheel"/>
@@ -76,5 +76,5 @@
     </gazebo>
     <!-- LEFT MID WHEEL LINK -->
-    <joint name="left_mid_wheel_joint" type="continuous">
+    <joint name="left_mid_wheel_joint" type="fixed">
         <parent link="base_link"/>
         <child link="left_mid_wheel"/>
@@ -102,5 +102,5 @@
     </gazebo>
     <!-- LEFT REAR WHEEL -->
-    <joint name="left_rear_wheel_joint" type="continuous">
+    <joint name="left_rear_wheel_joint" type="fixed">
         <parent link="base_link"/>
         <child link="left_rear_wheel"/>
@@ -128,5 +128,5 @@
     </gazebo>
     <!-- RIGHT FRONT WHEEL LINK -->
-    <joint name="right_front_wheel_joint" type="continuous">
+    <joint name="right_front_wheel_joint" type="fixed">
         <parent link="base_link"/>
         <child link="right_front_wheel"/>
@@ -154,5 +154,5 @@
     </gazebo>
     <!-- RIGHT MID WHEEL LINK -->
-    <joint name="right_mid_wheel_joint" type="continuous">
+    <joint name="right_mid_wheel_joint" type="fixed">
         <parent link="base_link"/>
         <child link="right_mid_wheel"/>
@@ -180,5 +180,5 @@
     </gazebo>
     <!-- RIGHT REAR WHEEL LINK -->
-    <joint name="right_rear_wheel_joint" type="continuous">
+    <joint name="right_rear_wheel_joint" type="fixed">
         <parent link="base_link"/>
         <child link="right_rear_wheel"/>
